Commit message: collision mailslot v1.0

File: project_starter_code/mmp_panda_new.urdf (robot description, URDF)
Before this commit: robot mmp_panda, 13 links, 12 joints
Links:
- link base_link: geometry collision box size=0.02 0.1 0.1; collision box size=0.02 0.1 0.1
- link leftfinger: geometry visual mesh filename=../../../model/panda/meshes/visual/finger.obj
- link rightfinger: geometry visual mesh filename=../../../model/panda/meshes/visual/finger.obj
