Commit message: add mobile base to world

File: project_starter_code/mmp_panda.urdf (robot description, URDF)
Before this commit: robot mmp_panda, 11 links, 10 joints
Links:
- link base_link: geometry visual mesh filename=../../../model/project_models/mailtruck.obj

Commit message: first couple states work

File: project_starter_code/mmp_panda.urdf (robot description, URDF)
Before this commit: robot mmp_panda, 11 links, 10 joints
Links:
- link base_link: mass 64.6 -> 10000

Commit message: added max velocity for truck

File: project_starter_code/mmp_panda.urdf (robot description, URDF)
Before this commit: robot mmp_panda, 11 links, 10 joints
Links:
- link base_link: mass 10000 -> 1000

Commit message: added functional gripper

File: project_starter_code/mmp_panda.urdf (robot description, URDF)
Before this commit: robot mmp_panda, 11 links, 10 joints
Links:
- added link leftfinger, mass 0.1; visual mesh filename=../../../model/panda/meshes/visual/finger.obj
- added link rightfinger, mass 0.1; visual mesh filename=../../../model/panda/meshes/visual/finger.obj
- link link7: mass 3.0 -> 1.8; geometry visual mesh filename=../../../model/panda/meshes/visual/hand.obj; visual mesh filename=../../../model/panda/meshes/visual/link7.obj
Joints:
- added joint finger_joint1: type prismatic, parent link7, child leftfinger, origin xyz=0 0 0.1654 rpy=0 0 -0.78539816339, axis 0 1 0, limit lower=0.0 upper=0.04 effort=20 velocity=0.2
- added joint finger_joint2: type prismatic, parent link7, child rightfinger, origin xyz=0 0 0.1654 rpy=0 0 -0.78539816339, axis 0 1 0, limit lower=0.0 upper=0.04 effort=20 velocity=0.2

Commit message: add mailslot and attempt to sim letter

File: project_starter_code/mmp_panda.urdf (robot description, URDF)
Before this commit: robot mmp_panda, 13 links, 12 joints
Links:
- link base_link: geometry collision mesh filename=../../../model/project_models/mailslot.obj; visual mesh filename=../../../model/project_models/mailslot.obj

Commit message: added mailbox collision

File: project_starter_code/mmp_panda.urdf (robot description, URDF)
Before this commit: robot mmp_panda, 13 links, 12 joints
Links:
- link leftfinger: geometry collision mesh filename=../../../model/panda/meshes/collision/finger.obj; visual mesh filename=../../../model/panda/meshes/visual/finger.obj
- link rightfinger: geometry collision mesh filename=../../../model/panda/meshes/collision/finger.obj; visual mesh filename=../../../model/panda/meshes/visual/finger.obj

Commit message: fixed gripper, added states, cleaned up code

File: project_starter_code/mmp_panda.urdf (robot description, URDF)
Before this commit: robot mmp_panda, 13 links, 12 joints
Links:
- link base_link: geometry visual box size=0.02 0.1 0.1; visual box size=0.02 0.1 0.1

Commit message: functional mail delivery

File: project_starter_code/mmp_panda.urdf (robot description, URDF)
Before this commit: robot mmp_panda, 13 links, 12 joints
Links:
- link base_link: geometry collision box size=0.18 0.3 0.02; visual mesh filename=../../../model/project_models/mailtruck.obj
